Commit message: first commit

File: articubot_one/description/face.xacro (robot description, xacro)
@@ -4,31 +4,14 @@
         <parent link="chassis"/>
         <child link="face_link"/>
-        <origin xyz="${chassis_length} 0 ${chassis_height/2}" rpy="0 0 0"/>
+        <origin xyz="0.4268 0 0.155" rpy="0 0 0"/>
     </joint>
     <link name="face_link">
         <visual>
-            <origin xyz="0 0.05 0.01" rpy="0 ${pi/2} 0"/>
+            <origin xyz="-0.011 0 -0.00" rpy="0 0 0"/>
             <geometry>
-                <cylinder radius="0.01" length="0.002"/>
+                <box size="0.0255 0.09 0.025"/>
             </geometry>
             <material name="black"/>
         </visual>
-        <visual>
-            <origin xyz="0 -0.05 0.01" rpy="0 ${pi/2} 0"/>
-            <geometry>
-                <cylinder radius="0.01" length="0.002"/>
-            </geometry>
-            <material name="black"/>
-        </visual>
-        <visual>
-            <origin xyz="-0.011 0 -0.00" rpy="0 ${1.5} 0"/>
-            <geometry>
-                <cylinder radius="0.05" length="0.02"/>
-            </geometry>
-            <material name="red"/>
-        </visual>
     </link>
-    <gazebo reference="face_link">
-        <material>Gazebo/Black</material>
-    </gazebo>
 </robot>

File: articubot_one/description/gazebo_control.xacro (robot description, xacro)
@@ -6,5 +6,5 @@
             <left_joint>left_wheel_joint</left_joint>
             <right_joint>right_wheel_joint</right_joint>
-            <wheel_separation>0.297</wheel_separation>
+            <wheel_separation>0.215</wheel_separation>
             <wheel_diameter>0.066</wheel_diameter>
             <!-- Limits -->

File: articubot_one/description/lidar.xacro (robot description, xacro)
@@ -4,10 +4,10 @@
         <parent link="chassis"/>
         <child link="laser_frame"/>
-        <origin xyz="0.122 0 0.212" rpy="0 0 0"/>
+        <origin xyz="0.04 0 0.27" rpy="0 0 0"/>
     </joint>
     <link name="laser_frame">
         <visual>
             <geometry>
-                <cylinder radius="0.05" length="0.04"/>
+                <cylinder radius="0.025" length="0.04"/>
             </geometry>
             <material name="black"/>
@@ -22,5 +22,5 @@
         <collision>
             <geometry>
-                <cylinder radius="0.05" length="0.04"/>
+                <cylinder radius="0.025" length="0.04"/>
             </geometry>
         </collision>
@@ -29,9 +29,37 @@
         </xacro:inertial_cylinder>
     </link>
-    <gazebo reference="laser_frame">
+    <joint name="ydlidar1_joint" type="fixed">
+        <parent link="chassis"/>
+        <child link="ydlidar1"/>
+        <origin xyz="0.0237 0.09876 0.268" rpy="0 0 0"/>
+    </joint>
+    <link name="ydlidar1">
+        <visual>
+            <origin xyz="0 0 -0.01" rpy="0 0 0"/>
+            <geometry>
+                <cylinder radius="0.018" length="0.034"/>
+            </geometry>
+            <material name="black"/>
+        </visual>
+    </link>
+    <joint name="ydlidar2_joint" type="fixed">
+        <parent link="chassis"/>
+        <child link="ydlidar2"/>
+        <origin xyz="0.3831 -0.09876 0.268" rpy="0 0 0"/>
+    </joint>
+    <link name="ydlidar2">
+        <visual>
+            <origin xyz="0 0 -0.01" rpy="0 0 0"/>
+            <geometry>
+                <cylinder radius="0.018" length="0.034"/>
+            </geometry>
+            <material name="black"/>
+        </visual>
+    </link>
+    <gazebo reference="ydlidar1">
         <material>Gazebo/Black</material>
-        <sensor name="laser" type="ray">
+        <sensor name="ydlidar1" type="ray">
             <pose> 0 0 0 0 0 0 </pose>
-            <visualize>false</visualize>
+            <visualize>true</visualize>
             <update_rate>10</update_rate>
             <ray>
@@ -48,10 +76,38 @@
                 </range>
             </ray>
-            <plugin name="laser_controller" filename="libgazebo_ros_ray_sensor.so">
+            <plugin name="laser_controller1" filename="libgazebo_ros_ray_sensor.so">
                 <ros>
-                    <argument>~/out:=scan</argument>
+                    <argument>~/out:=scan1</argument>
                 </ros>
                 <output_type>sensor_msgs/LaserScan</output_type>
-                <frame_name>laser_frame</frame_name>
+                <frame_name>ydlidar1</frame_name>
+            </plugin>
+        </sensor>
+    </gazebo>
+    <gazebo reference="ydlidar2">
+        <material>Gazebo/Black</material>
+        <sensor name="ydlidar2" type="ray">
+            <pose> 0 0 0 0 0 0 </pose>
+            <visualize>true</visualize>
+            <update_rate>10</update_rate>
+            <ray>
+                <scan>
+                    <horizontal>
+                        <samples>360</samples>
+                        <min_angle>-3.14</min_angle>
+                        <max_angle>3.14</max_angle>
+                    </horizontal>
+                </scan>
+                <range>
+                    <min>0.3</min>
+                    <max>12</max>
+                </range>
+            </ray>
+            <plugin name="laser_controller2" filename="libgazebo_ros_ray_sensor.so">
+                <ros>
+                    <argument>~/out:=scan2</argument>
+                </ros>
+                <output_type>sensor_msgs/LaserScan</output_type>
+                <frame_name>ydlidar2</frame_name>
             </plugin>
         </sensor>

File: articubot_one/description/robot_core.xacro (robot description, xacro)
@@ -2,16 +2,16 @@
 <robot xmlns:xacro="http://www.ros.org/wiki/xacro" >
     <xacro:include filename="inertial_macros.xacro"/>
-    <xacro:property name="chassis_length" value="0.335"/>
-    <xacro:property name="chassis_width" value="0.265"/>
-    <xacro:property name="chassis_height" value="0.138"/>
-    <xacro:property name="chassis_mass" value="1.0"/>
-    <xacro:property name="wheel_radius" value="0.065"/>
-    <xacro:property name="wheel_thickness" value="0.026"/>
-    <xacro:property name="wheel_mass" value="0.05"/>
-    <xacro:property name="wheel_offset_x" value="0.226"/>
-    <xacro:property name="wheel_offset_y" value="0.2085"/>
-    <xacro:property name="wheel_offset_z" value="0.01"/>
-    <xacro:property name="caster_wheel_radius" value="0.01"/>
-    <xacro:property name="caster_wheel_mass" value="0.01"/>
+    <xacro:property name="chassis_length" value="0.4068"/>
+    <xacro:property name="chassis_width" value="0.250"/>
+    <xacro:property name="chassis_height" value="0.24"/>
+    <xacro:property name="chassis_mass" value="10.0"/>
+    <xacro:property name="wheel_radius" value="0.066"/>
+    <xacro:property name="wheel_thickness" value="0.020"/>
+    <xacro:property name="wheel_mass" value="1.0"/>
+    <xacro:property name="wheel_offset_x" value="0.2034"/>
+    <xacro:property name="wheel_offset_y" value="0.1125"/>
+    <xacro:property name="wheel_offset_z" value="0.0495"/>
+    <xacro:property name="caster_wheel_radius" value="0.0175"/>
+    <xacro:property name="caster_wheel_mass" value="0.1"/>
     <xacro:property name="caster_wheel_offset_x" value="0.075"/>
     <xacro:property name="caster_wheel_offset_z" value="${wheel_offset_z - wheel_radius + caster_wheel_radius}"/>
@@ -75,4 +75,5 @@
         <origin xyz="0 ${wheel_offset_y} 0" rpy="-${pi/2} 0 0" />
         <axis xyz="0 0 1"/>
+        <joint_properties damping="0.0" friction="0.0" stiffness="0.1"/>
     </joint>
     <link name="left_wheel">
@@ -101,4 +102,5 @@
         <origin xyz="0 ${-wheel_offset_y} 0" rpy="${pi/2} 0 0" />
         <axis xyz="0 0 -1"/>
+    <joint_properties damping="0.0" friction="0.0" stiffness="0.1"/>
     </joint>
     <link name="right_wheel">
@@ -122,10 +124,73 @@
     </gazebo>
     <!-- CASTER WHEEL LINK -->
-    <joint name="caster_wheel_joint" type="fixed">
-        <parent link="chassis"/>
-        <child link="caster_wheel"/>
-        <origin xyz="${caster_wheel_offset_x} 0 ${caster_wheel_offset_z}"/>
-    </joint>
-    <link name="caster_wheel">
+    <joint name="caster_wheel_joint1" type="fixed">
+        <parent link="chassis"/>
+        <child link="caster_wheel1"/>
+        <origin xyz="0.0494 0.0565 0.0025"/>
+    </joint>
+    <joint name="caster_wheel_joint2" type="fixed">
+        <parent link="chassis"/>
+        <child link="caster_wheel2"/>
+        <origin xyz="0.0494 -0.0565 0.0025"/>
+    </joint>
+    <joint name="caster_wheel_joint3" type="fixed">
+        <parent link="chassis"/>
+        <child link="caster_wheel3"/>
+        <origin xyz="0.3554 0.0565 0.0025"/>
+    </joint>
+    <joint name="caster_wheel_joint4" type="fixed">
+        <parent link="chassis"/>
+        <child link="caster_wheel4"/>
+        <origin xyz="0.3554 -0.0565 0.0025"/>
+    </joint>
+    <link name="caster_wheel1">
+        <visual>
+            <geometry>
+                <sphere radius="${caster_wheel_radius}"/>
+            </geometry>
+            <material name="white"/>
+        </visual>
+        <collision>
+            <geometry>
+                <sphere radius="${caster_wheel_radius}"/>
+            </geometry>
+        </collision>
+        <xacro:inertial_sphere mass="${caster_wheel_mass}" radius="${caster_wheel_radius}">
+            <origin xyz="0 0 0" rpy="0 0 0"/>
+        </xacro:inertial_sphere>
+    </link>
+    <link name="caster_wheel2">
+        <visual>
+            <geometry>
+                <sphere radius="${caster_wheel_radius}"/>
+            </geometry>
+            <material name="white"/>
+        </visual>
+        <collision>
+            <geometry>
+                <sphere radius="${caster_wheel_radius}"/>
+            </geometry>
+        </collision>
+        <xacro:inertial_sphere mass="${caster_wheel_mass}" radius="${caster_wheel_radius}">
+            <origin xyz="0 0 0" rpy="0 0 0"/>
+        </xacro:inertial_sphere>
+    </link>
+    <link name="caster_wheel3">
+        <visual>
+            <geometry>
+                <sphere radius="${caster_wheel_radius}"/>
+            </geometry>
+            <material name="white"/>
+        </visual>
+        <collision>
+            <geometry>
+                <sphere radius="${caster_wheel_radius}"/>
+            </geometry>
+        </collision>
+        <xacro:inertial_sphere mass="${caster_wheel_mass}" radius="${caster_wheel_radius}">
+            <origin xyz="0 0 0" rpy="0 0 0"/>
+        </xacro:inertial_sphere>
+    </link>
+    <link name="caster_wheel4">
         <visual>
             <geometry>
