Commit message: fixed jumping corridor

File: articubot_one/description/robot_core.xacro (robot description, xacro)
@@ -14,5 +14,5 @@
     <xacro:property name="caster_wheel_radius" value="0.0175"/>
     <xacro:property name="caster_wheel_mass" value="0.1"/>
-    <xacro:property name="caster_wheel_offset_x" value="0.075"/>
+    <xacro:property name="caster_wheel_offset_x" value="0.073"/>
     <xacro:property name="caster_wheel_offset_z" value="${wheel_offset_z - wheel_radius + caster_wheel_radius}"/>
     <material name="white">

File: articubot_one/description/ros2_control.xacro (robot description, xacro)
@@ -11,5 +11,5 @@
                 <param name="baud_rate">57600</param>
                 <param name="timeout">1000</param>
-                <param name="enc_counts_per_rev">400</param>
+                <param name="enc_counts_per_rev">92800</param>
             </hardware>
             <joint name="left_wheel_joint">

Commit message: improvements the turning

File: articubot_one/description/robot_core.xacro (robot description, xacro)
@@ -11,5 +11,5 @@
     <xacro:property name="wheel_offset_x" value="0.2034"/>
     <xacro:property name="wheel_offset_y" value="0.1125"/>
-    <xacro:property name="wheel_offset_z" value="0.0490"/>
+    <xacro:property name="wheel_offset_z" value="0.050"/>
     <xacro:property name="caster_wheel_radius" value="0.0175"/>
     <xacro:property name="caster_wheel_mass" value="0.1"/>
@@ -89,4 +89,6 @@
     <gazebo reference="left_wheel">
         <material>Gazebo/Blue</material>
+        <mu1>10.0</mu1>
+        <mu2>10.0</mu2>
     </gazebo>
     <!-- RIGHT WHEEL LINK -->
@@ -116,4 +118,6 @@
     <gazebo reference="right_wheel">
         <material>Gazebo/Blue</material>
+        <mu1>10.0</mu1>
+        <mu2>10.0</mu2>
     </gazebo>
     <!-- CASTER WHEEL LINK -->
@@ -204,6 +208,6 @@
     <gazebo reference="caster_wheel">
         <material>Gazebo/White</material>
-        <mu1 value="0.001"/>
-        <mu2 value="0.001"/>
+        <mu1>0.0</mu1>
+        <mu2>0.0</mu2>
     </gazebo>
 </robot>

Commit message: first commit

File: articubot_one/description/robot_core.xacro (robot description, xacro)
@@ -59,5 +59,5 @@
             <origin xyz="${chassis_length/2} 0 ${chassis_height/2}"/>
             <geometry>
-                <box size="${chassis_length} ${chassis_width} ${chassis_height/5}"/>
+                <box size="${chassis_length} ${chassis_width} ${chassis_height}"/>
             </geometry>
             <material name="orange"/>
