Commit message: slam with 2 lasers and world options

File: articubot_one/description/lidar.xacro (robot description, xacro)
@@ -46,5 +46,5 @@
         <parent link="chassis"/>
         <child link="ydlidar2"/>
-        <origin xyz="0.3831 -0.09876 0.268" rpy="0 0 0"/>
+        <origin xyz="0.3831 -0.09876 0.358" rpy="0 0 0"/>
     </joint>
     <link name="ydlidar2">

Commit message: enable ekf on nuc

File: articubot_one/description/lidar.xacro (robot description, xacro)
@@ -29,4 +29,5 @@
         </xacro:inertial_cylinder>
     </link>
+<!--
     <joint name="ydlidar1_joint" type="fixed">
         <parent link="chassis"/>
@@ -57,4 +58,34 @@
         </visual>
     </link>
+ -->
+    <gazebo reference="laser_frame">
+        <material>Gazebo/Black</material>
+        <sensor name="sensor" type="ray">
+            <pose> 0 0 0 0 0 0 </pose>
+            <visualize>true</visualize>
+            <update_rate>10</update_rate>
+            <ray>
+                <scan>
+                    <horizontal>
+                        <samples>360</samples>
+                        <min_angle>-3.14</min_angle>
+                        <max_angle>3.14</max_angle>
+                    </horizontal>
+                </scan>
+                <range>
+                    <min>0.3</min>
+                    <max>12</max>
+                </range>
+            </ray>
+            <plugin name="laser_controller" filename="libgazebo_ros_ray_sensor.so">
+                <ros>
+                    <argument>~/out:=scan</argument>
+                </ros>
+                <output_type>sensor_msgs/LaserScan</output_type>
+                <frame_name>laser_frame</frame_name>
+            </plugin>
+        </sensor>
+    </gazebo>
+<!--
     <gazebo reference="ydlidar1">
         <material>Gazebo/Black</material>
@@ -113,3 +144,4 @@
         </sensor>
     </gazebo>
+     -->
 </robot>

Commit message: bno055 imu update

File: articubot_one/description/lidar.xacro (robot description, xacro)
@@ -7,4 +7,32 @@
     </joint>
     <link name="laser_frame">
+        <visual>
+            <geometry>
+                <cylinder radius="0.025" length="0.04"/>
+            </geometry>
+            <material name="black"/>
+        </visual>
+        <visual>
+            <origin xyz="0 0 -0.05"/>
+            <geometry>
+                <cylinder radius="0.01" length="0.1"/>
+            </geometry>
+            <material name="black"/>
+        </visual>
+        <collision>
+            <geometry>
+                <cylinder radius="0.025" length="0.04"/>
+            </geometry>
+        </collision>
+        <xacro:inertial_cylinder mass="0.1" length="0.04" radius="0.05">
+            <origin xyz="0 0 0" rpy="0 0 0"/>
+        </xacro:inertial_cylinder>
+    </link>
+    <joint name="bno055_joint" type="fixed">
+        <parent link="chassis"/>
+        <child link="bno055"/>
+        <origin xyz="0.2 0 0.20" rpy="0 0 0"/>
+    </joint>
+    <link name="bno055">
         <visual>
             <geometry>

Commit message: minor fix

File: articubot_one/description/lidar.xacro (robot description, xacro)
@@ -1,5 +1,5 @@
 <?xml version="1.0"?>
 <robot xmlns:xacro="http://www.ros.org/wiki/xacro" >
-    <joint name="laser_joint" type="fixed">
+    <!-- <joint name="laser_joint" type="fixed">
         <parent link="chassis"/>
         <child link="laser_frame"/>
@@ -28,5 +28,5 @@
             <origin xyz="0 0 0" rpy="0 0 0"/>
         </xacro:inertial_cylinder>
-    </link>
+    </link> -->
     <joint name="ydlidar1_joint" type="fixed">
         <parent link="chassis"/>
@@ -72,6 +72,6 @@
                 </scan>
                 <range>
-                    <min>0.3</min>
-                    <max>12</max>
+                    <min>0.03</min>
+                    <max>30</max>
                 </range>
             </ray>
@@ -100,6 +100,6 @@
                 </scan>
                 <range>
-                    <min>0.3</min>
-                    <max>12</max>
+                    <min>0.03</min>
+                    <max>30</max>
                 </range>
             </ray>

Commit message: ready for real

File: articubot_one/description/lidar.xacro (robot description, xacro)
@@ -32,5 +32,5 @@
         <parent link="chassis"/>
         <child link="ydlidar1"/>
-        <origin xyz="0.0237 0.09876 0.268" rpy="0 0 0"/>
+        <origin xyz="0.0237 0.0 0.268" rpy="0 0 0"/>
     </joint>
     <link name="ydlidar1">
@@ -46,5 +46,5 @@
         <parent link="chassis"/>
         <child link="ydlidar2"/>
-        <origin xyz="0.3831 -0.09876 0.358" rpy="0 0 0"/>
+        <origin xyz="0.3831 0.0 0.358" rpy="0 0 0"/>
     </joint>
     <link name="ydlidar2">

Commit message: laser filter

File: articubot_one/description/lidar.xacro (robot description, xacro)
@@ -32,5 +32,6 @@
         <parent link="chassis"/>
         <child link="ydlidar1"/>
-        <origin xyz="0.0237 0.0 0.268" rpy="0 0 0"/>
+        <origin xyz="0.0037 0.0 0.268" rpy="0 0 -1.57"/>
+        <!-- <origin xyz="0.0237 0.0 0.268" rpy="0 0 0"/> -->
     </joint>
     <link name="ydlidar1">
@@ -46,5 +47,6 @@
         <parent link="chassis"/>
         <child link="ydlidar2"/>
-        <origin xyz="0.3831 0.0 0.358" rpy="0 0 0"/>
+        <origin xyz="0.4031 0.0 0.358" rpy="0 0 1.57"/>
+        <!-- <origin xyz="0.3831 0.0 0.358" rpy="0 0 0"/> -->
     </joint>
     <link name="ydlidar2">

Commit message: set lidar location

File: articubot_one/description/lidar.xacro (robot description, xacro)
@@ -1,8 +1,8 @@
 <?xml version="1.0"?>
 <robot xmlns:xacro="http://www.ros.org/wiki/xacro" >
-    <!-- <joint name="laser_joint" type="fixed">
+    <joint name="laser_joint" type="fixed">
         <parent link="chassis"/>
         <child link="laser_frame"/>
-        <origin xyz="0.04 0 0.27" rpy="0 0 0"/>
+        <origin xyz="0.21 0 0.27" rpy="0 0 0"/>
     </joint>
     <link name="laser_frame">
@@ -28,10 +28,11 @@
             <origin xyz="0 0 0" rpy="0 0 0"/>
         </xacro:inertial_cylinder>
-    </link> -->
-    <joint name="ydlidar1_joint" type="fixed">
+    </link>
+<!--
+     <joint name="ydlidar1_joint" type="fixed">
         <parent link="chassis"/>
         <child link="ydlidar1"/>
         <origin xyz="0.0037 0.0 0.268" rpy="0 0 -1.57"/>
-        <!-- <origin xyz="0.0237 0.0 0.268" rpy="0 0 0"/> -->
+        <origin xyz="0.0237 0.0 0.268" rpy="0 0 0"/>
     </joint>
     <link name="ydlidar1">
@@ -48,5 +49,4 @@
         <child link="ydlidar2"/>
         <origin xyz="0.4031 0.0 0.358" rpy="0 0 1.57"/>
-        <!-- <origin xyz="0.3831 0.0 0.358" rpy="0 0 0"/> -->
     </joint>
     <link name="ydlidar2">
@@ -115,3 +115,4 @@
         </sensor>
     </gazebo>
+      -->
 </robot>

Commit message: edit frame name

File: articubot_one/description/lidar.xacro (robot description, xacro)
@@ -1,6 +1,6 @@
 <?xml version="1.0"?>
 <robot xmlns:xacro="http://www.ros.org/wiki/xacro" >
-    <!-- <joint name="laser_joint" type="fixed">
-        <parent link="chassis"/>
+    <joint name="laser_joint" type="fixed">
+        <parent link="base_link_frame"/>
         <child link="laser_frame"/>
         <origin xyz="0.04 0 0.27" rpy="0 0 0"/>
@@ -28,6 +28,6 @@
             <origin xyz="0 0 0" rpy="0 0 0"/>
         </xacro:inertial_cylinder>
-    </link> -->
-    <joint name="ydlidar1_joint" type="fixed">
+    </link>
+    <!-- <joint name="ydlidar1_joint" type="fixed">
         <parent link="chassis"/>
         <child link="ydlidar1"/>
@@ -113,3 +113,4 @@
         </sensor>
     </gazebo>
+     -->
 </robot>

File: articubot_one/description/robot_core.xacro (robot description, xacro)
@@ -32,9 +32,9 @@
     </material>
     <!-- BASE LINK -->
-    <link name="base_link">
+    <link name="base_link_frame">
     </link>
     <!-- BASE_FOOTPRINT LINK -->
     <joint name="base_footprint_joint" type="fixed">
-        <parent link="base_link"/>
+        <parent link="base_link_frame"/>
         <child link="base_footprint"/>
         <origin xyz="0 0 0" rpy="0 0 0"/>
@@ -44,5 +44,5 @@
     <!-- CHASSIS LINK -->
     <joint name="chassis_joint" type="fixed">
-        <parent link="base_link"/>
+        <parent link="base_link_frame"/>
         <child link="chassis"/>
         <origin xyz="${-wheel_offset_x} 0 ${-wheel_offset_z}"/>
@@ -71,5 +71,5 @@
     <!-- LEFT WHEEL LINK -->
     <joint name="left_wheel_joint" type="continuous">
-        <parent link="base_link"/>
+        <parent link="base_link_frame"/>
         <child link="left_wheel"/>
         <origin xyz="0 ${wheel_offset_y} 0" rpy="-${pi/2} 0 0" />
@@ -98,5 +98,5 @@
     <!-- RIGHT WHEEL LINK -->
     <joint name="right_wheel_joint" type="continuous">
-        <parent link="base_link"/>
+        <parent link="base_link_frame"/>
         <child link="right_wheel"/>
         <origin xyz="0 ${-wheel_offset_y} 0" rpy="${pi/2} 0 0" />

Commit message: nav without slam_toolbox but no costmap

File: articubot_one/description/lidar.xacro (robot description, xacro)
@@ -1,5 +1,5 @@
 <?xml version="1.0"?>
 <robot xmlns:xacro="http://www.ros.org/wiki/xacro" >
-    <!-- <joint name="laser_joint" type="fixed">
+    <joint name="laser_joint" type="fixed">
         <parent link="chassis"/>
         <child link="laser_frame"/>
@@ -28,10 +28,10 @@
             <origin xyz="0 0 0" rpy="0 0 0"/>
         </xacro:inertial_cylinder>
-    </link> -->
-    <joint name="ydlidar1_joint" type="fixed">
+    </link>
+    <!-- <joint name="ydlidar1_joint" type="fixed">
         <parent link="chassis"/>
         <child link="ydlidar1"/>
         <origin xyz="0.0037 0.0 0.268" rpy="0 0 -1.57"/>
-        <!-- <origin xyz="0.0237 0.0 0.268" rpy="0 0 0"/> -->
+    <origin xyz="0.0237 0.0 0.268" rpy="0 0 0"/>
     </joint>
     <link name="ydlidar1">
@@ -48,5 +48,5 @@
         <child link="ydlidar2"/>
         <origin xyz="0.4031 0.0 0.358" rpy="0 0 1.57"/>
-        <!-- <origin xyz="0.3831 0.0 0.358" rpy="0 0 0"/> -->
+        <origin xyz="0.3831 0.0 0.358" rpy="0 0 0"/>
     </joint>
     <link name="ydlidar2">
@@ -115,3 +115,4 @@
         </sensor>
     </gazebo>
+     -->
 </robot>

Commit message: works simuation

File: articubot_one/description/lidar.xacro (robot description, xacro)
@@ -1,8 +1,8 @@
 <?xml version="1.0"?>
 <robot xmlns:xacro="http://www.ros.org/wiki/xacro" >
-    <!-- <joint name="laser_joint" type="fixed">
+    <joint name="laser_joint" type="fixed">
         <parent link="chassis"/>
         <child link="laser_frame"/>
-        <origin xyz="0.04 0 0.27" rpy="0 0 0"/>
+        <origin xyz="0.10 0 0.55" rpy="0 0 0"/>
     </joint>
     <link name="laser_frame">
@@ -13,25 +13,41 @@
             <material name="black"/>
         </visual>
-        <visual>
-            <origin xyz="0 0 -0.05"/>
-            <geometry>
-                <cylinder radius="0.01" length="0.1"/>
-            </geometry>
-            <material name="black"/>
-        </visual>
-        <collision>
-            <geometry>
-                <cylinder radius="0.025" length="0.04"/>
-            </geometry>
-        </collision>
         <xacro:inertial_cylinder mass="0.1" length="0.04" radius="0.05">
             <origin xyz="0 0 0" rpy="0 0 0"/>
         </xacro:inertial_cylinder>
-    </link> -->
-    <joint name="ydlidar1_joint" type="fixed">
+    </link>
+  <gazebo reference="laser_frame">
+        <material>Gazebo/Black</material>
+        <sensor name="laser" type="ray">
+            <pose> 0 0 0 0 0 0 </pose>
+            <visualize>false</visualize>
+            <update_rate>10</update_rate>
+            <ray>
+                <scan>
+                    <horizontal>
+                        <samples>360</samples>
+                        <min_angle>-3.14</min_angle>
+                        <max_angle>3.14</max_angle>
+                    </horizontal>
+                </scan>
+                <range>
+                    <min>0.03</min>
+                    <max>30</max>
+                </range>
+            </ray>
+            <plugin name="laser" filename="libgazebo_ros_ray_sensor.so">
+                <ros>
+                    <argument>~/out:=scan</argument>
+                </ros>
+                <output_type>sensor_msgs/LaserScan</output_type>
+                <frame_name>laser_frame</frame_name>
+            </plugin>
+        </sensor>
+    </gazebo>
+    <!-- <joint name="ydlidar1_joint" type="fixed">
         <parent link="chassis"/>
         <child link="ydlidar1"/>
         <origin xyz="0.0037 0.0 0.268" rpy="0 0 -1.57"/>
-        <!-- <origin xyz="0.0237 0.0 0.268" rpy="0 0 0"/> -->
+         <origin xyz="0.0237 0.0 0.268" rpy="0 0 0"/>
     </joint>
     <link name="ydlidar1">
@@ -48,5 +64,5 @@
         <child link="ydlidar2"/>
         <origin xyz="0.4031 0.0 0.358" rpy="0 0 1.57"/>
-        <!-- <origin xyz="0.3831 0.0 0.358" rpy="0 0 0"/> -->
+         <origin xyz="0.3831 0.0 0.358" rpy="0 0 0"/>
     </joint>
     <link name="ydlidar2">
@@ -115,3 +131,4 @@
         </sensor>
     </gazebo>
+     -->
 </robot>

Commit message: first commit

File: articubot_one/description/lidar.xacro (robot description, xacro)
@@ -4,5 +4,5 @@
         <parent link="chassis"/>
         <child link="laser_frame"/>
-        <origin xyz="0.10 0 0.55" rpy="0 0 0"/>
+        <origin xyz="0.10 0 0.30" rpy="0 0 0"/>
     </joint>
     <link name="laser_frame">
@@ -33,5 +33,5 @@
                 <range>
                     <min>0.03</min>
-                    <max>30</max>
+                    <max>40</max>
                 </range>
             </ray>

File: articubot_one/description/robot_core.xacro (robot description, xacro)
@@ -11,5 +11,5 @@
     <xacro:property name="wheel_offset_x" value="0.2034"/>
     <xacro:property name="wheel_offset_y" value="0.1125"/>
-    <xacro:property name="wheel_offset_z" value="0.0495"/>
+    <xacro:property name="wheel_offset_z" value="0.0490"/>
     <xacro:property name="caster_wheel_radius" value="0.0175"/>
     <xacro:property name="caster_wheel_mass" value="0.1"/>
@@ -56,10 +56,4 @@
             <material name="orange"/>
         </visual>
-        <collision>
-            <origin xyz="${chassis_length/2} 0 ${chassis_height/2}"/>
-            <geometry>
-                <box size="${chassis_length} ${chassis_width} ${chassis_height}"/>
-            </geometry>
-        </collision>
         <xacro:inertial_box mass="0.5" x="${chassis_length}" y="${chassis_width}" z="${chassis_height}">
             <origin xyz="${chassis_length/2} 0 ${chassis_height/2}" rpy="0 0 0"/>

Commit message: new uber map

File: articubot_one/description/lidar.xacro (robot description, xacro)
@@ -4,5 +4,5 @@
         <parent link="chassis"/>
         <child link="laser_frame"/>
-        <origin xyz="0.10 0 0.30" rpy="0 0 0"/>
+        <origin xyz="0.10 0 0.40" rpy="0 0 0"/>
     </joint>
     <link name="laser_frame">
@@ -32,5 +32,5 @@
                 </scan>
                 <range>
-                    <min>0.03</min>
+                    <min>0.17</min>
                     <max>40</max>
                 </range>

File: articubot_one/description/robot_core.xacro (robot description, xacro)
@@ -56,4 +56,11 @@
             <material name="orange"/>
         </visual>
+        <collision>
+            <origin xyz="${chassis_length/2} 0 ${chassis_height/2}"/>
+            <geometry>
+                <box size="${chassis_length} ${chassis_width} ${chassis_height/5}"/>
+            </geometry>
+            <material name="orange"/>
+        </collision>
         <xacro:inertial_box mass="0.5" x="${chassis_length}" y="${chassis_width}" z="${chassis_height}">
             <origin xyz="${chassis_length/2} 0 ${chassis_height/2}" rpy="0 0 0"/>
@@ -80,5 +87,5 @@
         <collision>
             <geometry>
-                <sphere radius="${wheel_radius}"/>
+                <cylinder radius="${wheel_radius}" length="${wheel_thickness}"/>
             </geometry>
         </collision>
@@ -109,5 +116,5 @@
         <collision>
             <geometry>
-                <sphere radius="${wheel_radius}"/>
+                <cylinder radius="${wheel_radius}" length="${wheel_thickness}"/>
             </geometry>
         </collision>

Commit message: new branch

File: articubot_one/description/lidar.xacro (robot description, xacro)
@@ -2,5 +2,5 @@
 <robot xmlns:xacro="http://www.ros.org/wiki/xacro" >
     <joint name="laser_joint" type="fixed">
-        <parent link="base_link_frame"/>
+        <parent link="base_link"/>
         <child link="laser_frame"/>
         <origin xyz="0.04 0 0.27" rpy="0 0 0"/>

File: articubot_one/description/robot_core.xacro (robot description, xacro)
@@ -32,9 +32,9 @@
     </material>
     <!-- BASE LINK -->
-    <link name="base_link_frame">
+    <link name="base_link">
     </link>
     <!-- BASE_FOOTPRINT LINK -->
     <joint name="base_footprint_joint" type="fixed">
-        <parent link="base_link_frame"/>
+        <parent link="base_link"/>
         <child link="base_footprint"/>
         <origin xyz="0 0 0" rpy="0 0 0"/>
@@ -44,5 +44,5 @@
     <!-- CHASSIS LINK -->
     <joint name="chassis_joint" type="fixed">
-        <parent link="base_link_frame"/>
+        <parent link="base_link"/>
         <child link="chassis"/>
         <origin xyz="${-wheel_offset_x} 0 ${-wheel_offset_z}"/>
@@ -71,5 +71,5 @@
     <!-- LEFT WHEEL LINK -->
     <joint name="left_wheel_joint" type="continuous">
-        <parent link="base_link_frame"/>
+        <parent link="base_link"/>
         <child link="left_wheel"/>
         <origin xyz="0 ${wheel_offset_y} 0" rpy="-${pi/2} 0 0" />
@@ -98,5 +98,5 @@
     <!-- RIGHT WHEEL LINK -->
     <joint name="right_wheel_joint" type="continuous">
-        <parent link="base_link_frame"/>
+        <parent link="base_link"/>
         <child link="right_wheel"/>
         <origin xyz="0 ${-wheel_offset_y} 0" rpy="${pi/2} 0 0" />

File: articubot_one/description/ros2_control.xacro (robot description, xacro)
@@ -8,5 +8,5 @@
                 <param name="right_wheel_name">right_wheel_joint</param>
                 <param name="loop_rate">30</param>
-                <param name="device">/dev/serial/by-id/usb-1a86_USB_Serial-if00-port0</param>
+                <param name="device">/dev/ttyUSB0</param>
                 <param name="baud_rate">57600</param>
                 <param name="timeout">1000</param>
